Commit message: updating to add the kinova arm coupler

File: robotiq_85_description/urdf/robotiq_85_gripper.transmission.xacro (robot description, xacro)
@@ -1,11 +1,11 @@
 <?xml version="1.0"?>
-<robot xmlns:xacro="http://www.ros.org/wiki/xacro">
+<robot xmlns:xacro="http://ros.org/wiki/xacro">
   <xacro:macro name="robotiq_85_gripper_transmission" params="prefix">
-        <transmission name="${prefix}robotiq_85_left_knuckle_trans">
+        <transmission name="${prefix}gripper_finger1_trans">
             <type>transmission_interface/SimpleTransmission</type>
-            <joint name="${prefix}robotiq_85_left_knuckle_joint">
+            <joint name="${prefix}gripper_finger1_joint">
                 <hardwareInterface>PositionJointInterface</hardwareInterface>
             </joint>
-            <actuator name="${prefix}robotiq_85_left_knuckle_motor">
+            <actuator name="${prefix}gripper_finger1_motor">
                 <mechanicalReduction>1</mechanicalReduction>
                 <hardwareInterface>PositionJointInterface</hardwareInterface>
@@ -15,30 +15,30 @@
                 <!-- loading plugin: mimic joints works in gazebo now -->
             <plugin filename="libroboticsgroup_gazebo_mimic_joint_plugin.so" name="${prefix}mimic_robotiq_85_1">
-                <joint>${prefix}robotiq_85_left_knuckle_joint</joint>
-                <mimicJoint>${prefix}robotiq_85_right_knuckle_joint</mimicJoint>
+                <joint>${prefix}gripper_finger1_joint</joint>
+                <mimicJoint>${prefix}gripper_finger2_joint</mimicJoint>
                 <!--multiplier>1.0</multiplier>
                 <offset>0.0</offset-->
             </plugin>
             <plugin filename="libroboticsgroup_gazebo_mimic_joint_plugin.so" name="${prefix}mimic_robotiq_85_2">
-                <joint>${prefix}robotiq_85_left_knuckle_joint</joint>
-                <mimicJoint>${prefix}robotiq_85_left_inner_knuckle_joint</mimicJoint>
+                <joint>${prefix}gripper_finger1_joint</joint>
+                <mimicJoint>${prefix}gripper_finger2_inner_knuckle_joint</mimicJoint>
                 <!--multiplier>1.0</multiplier>
                 <offset>0.0</offset-->
             </plugin>
             <plugin filename="libroboticsgroup_gazebo_mimic_joint_plugin.so" name="${prefix}mimic_robotiq_85_3">
-                <joint>${prefix}robotiq_85_left_knuckle_joint</joint>
-                <mimicJoint>${prefix}robotiq_85_right_inner_knuckle_joint</mimicJoint>
+                <joint>${prefix}gripper_finger1_joint</joint>
+                <mimicJoint>${prefix}gripper_finger1_inner_knuckle_joint</mimicJoint>
                 <!--multiplier>1.0</multiplier>
                 <offset>0.0</offset-->
             </plugin>
             <plugin filename="libroboticsgroup_gazebo_mimic_joint_plugin.so" name="${prefix}mimic_robotiq_85_4">
-                <joint>${prefix}robotiq_85_left_knuckle_joint</joint>
-                <mimicJoint>${prefix}robotiq_85_left_finger_tip_joint</mimicJoint>
+                <joint>${prefix}gripper_finger1_joint</joint>
+                <mimicJoint>${prefix}gripper_finger1_finger_tip_joint</mimicJoint>
                 <multiplier>-1.0</multiplier>
                 <offset>0.0</offset>
             </plugin>
             <plugin filename="libroboticsgroup_gazebo_mimic_joint_plugin.so" name="${prefix}mimic_robotiq_85_5">
-                <joint>${prefix}robotiq_85_left_knuckle_joint</joint>
-                <mimicJoint>${prefix}robotiq_85_right_finger_tip_joint</mimicJoint>
+                <joint>${prefix}gripper_finger1_joint</joint>
+                <mimicJoint>${prefix}gripper_finger2_finger_tip_joint</mimicJoint>
                 <multiplier>-1.0</multiplier>
                 <offset>0.0</offset>

File: robotiq_85_description/urdf/robotiq_85_gripper.urdf.xacro (robot description, xacro)
@@ -2,12 +2,11 @@
 <robot name="robotiq_85_gripper" xmlns:xacro="http://ros.org/wiki/xacro">
     <xacro:include filename="$(find robotiq_85_description)/urdf/robotiq_85_gripper.transmission.xacro" />
-    <property name="pi" value="3.14159"/>
     <xacro:macro name="robotiq_85_gripper" params="prefix parent *origin">
-        <joint name="${prefix}robotiq_85_base_joint" type="fixed">
+        <joint name="${prefix}gripper_base_joint" type="fixed">
             <parent link="${parent}"/>
-            <child link="${prefix}robotiq_85_base_link"/>
+            <child link="${prefix}gripper_base_link"/>
             <xacro:insert_block name="origin"/>
         </joint>
-        <link name="${prefix}robotiq_85_base_link">
+        <link name="${prefix}gripper_base_link">
             <visual>
                 <geometry>
@@ -28,20 +27,27 @@
             </inertial>
         </link>
-        <joint name="${prefix}robotiq_85_left_knuckle_joint" type="revolute">
-            <parent link="${prefix}robotiq_85_base_link"/>
-            <child link="${prefix}robotiq_85_left_knuckle_link"/>
+        <gazebo reference="${prefix}gripper_base_link">
+            <implicitSpringDamper>1</implicitSpringDamper>
+            <mu1>100000</mu1>
+            <mu2>100000</mu2>
+            <kp>100000000.0</kp>
+            <kd>1.0</kd>
+        </gazebo>
+        <joint name="${prefix}gripper_finger1_joint" type="revolute">
+            <parent link="${prefix}gripper_base_link"/>
+            <child link="${prefix}gripper_finger1_knuckle_link"/>
             <axis xyz="0 0 1"/>
             <origin rpy="${pi} 0.0 0.0" xyz="0.05490451627 0.03060114443 0.0"/>
             <limit lower="0.0" upper="0.804" velocity="2.0" effort="1000"/>
         </joint>
-        <joint name="${prefix}robotiq_85_right_knuckle_joint" type="continuous">
-            <parent link="${prefix}robotiq_85_base_link"/>
-            <child link="${prefix}robotiq_85_right_knuckle_link"/>
+        <joint name="${prefix}gripper_finger2_joint" type="revolute">
+            <parent link="${prefix}gripper_base_link"/>
+            <child link="${prefix}gripper_finger2_knuckle_link"/>
             <axis xyz="0 0 1"/>
             <origin rpy="0.0 0.0 0.0" xyz="0.05490451627 -0.03060114443 0.0"/>
             <limit lower="-3.14" upper="3.14" velocity="100.0" effort="1000"/>
-            <mimic joint="${prefix}robotiq_85_left_knuckle_joint"/>
-        </joint>
-        <link name="${prefix}robotiq_85_left_knuckle_link">
+            <mimic joint="${prefix}gripper_finger1_joint"/>
+        </joint>
+        <link name="${prefix}gripper_finger1_knuckle_link">
             <visual>
                 <geometry>
@@ -62,5 +68,12 @@
             </inertial>
         </link>
-        <link name="${prefix}robotiq_85_right_knuckle_link">
+        <gazebo reference="${prefix}gripper_finger1_knuckle_link">
+            <implicitSpringDamper>1</implicitSpringDamper>
+            <mu1>100000</mu1>
+            <mu2>100000</mu2>
+            <kp>100000000.0</kp>
+            <kd>1.0</kd>
+        </gazebo>
+        <link name="${prefix}gripper_finger2_knuckle_link">
             <visual>
                 <geometry>
@@ -81,15 +94,22 @@
             </inertial>
         </link>
-        <joint name="${prefix}robotiq_85_left_finger_joint" type="fixed">
-            <parent link="${prefix}robotiq_85_left_knuckle_link"/>
-            <child link="${prefix}robotiq_85_left_finger_link"/>
+        <gazebo reference="${prefix}gripper_finger2_knuckle_link">
+            <implicitSpringDamper>1</implicitSpringDamper>
+            <mu1>100000</mu1>
+            <mu2>100000</mu2>
+            <kp>100000000.0</kp>
+            <kd>1.0</kd>
+        </gazebo>
+        <joint name="${prefix}gripper_finger1_finger_joint" type="fixed">
+            <parent link="${prefix}gripper_finger1_knuckle_link"/>
+            <child link="${prefix}gripper_finger1_finger_link"/>
             <origin xyz="-0.00408552455 -0.03148604435 0.0" rpy="0 0 0" />
         </joint>
-        <joint name="${prefix}robotiq_85_right_finger_joint" type="fixed">
-            <parent link="${prefix}robotiq_85_right_knuckle_link"/>
-            <child link="${prefix}robotiq_85_right_finger_link"/>
+        <joint name="${prefix}gripper_finger2_finger_joint" type="fixed">
+            <parent link="${prefix}gripper_finger2_knuckle_link"/>
+            <child link="${prefix}gripper_finger2_finger_link"/>
             <origin xyz="-0.00408552455 -0.03148604435 0.0" rpy="0 0 0" />
         </joint>
-        <link name="${prefix}robotiq_85_left_finger_link">
+        <link name="${prefix}gripper_finger1_finger_link">
             <visual>
                 <geometry>
@@ -110,5 +130,12 @@
             </inertial>
         </link>
-        <link name="${prefix}robotiq_85_right_finger_link">
+        <gazebo reference="${prefix}gripper_finger1_finger_link">
+            <implicitSpringDamper>1</implicitSpringDamper>
+            <mu1>100000</mu1>
+            <mu2>100000</mu2>
+            <kp>100000000.0</kp>
+            <kd>1.0</kd>
+        </gazebo>
+        <link name="${prefix}gripper_finger2_finger_link">
             <visual>
                 <geometry>
@@ -129,21 +156,28 @@
             </inertial>
         </link>
-        <joint name="${prefix}robotiq_85_left_inner_knuckle_joint" type="continuous">
-            <parent link="${prefix}robotiq_85_base_link"/>
-            <child link="${prefix}robotiq_85_left_inner_knuckle_link"/>
+        <gazebo reference="${prefix}gripper_finger2_finger_link">
+            <implicitSpringDamper>1</implicitSpringDamper>
+            <mu1>100000</mu1>
+            <mu2>100000</mu2>
+            <kp>100000000.0</kp>
+            <kd>1.0</kd>
+        </gazebo>
+        <joint name="${prefix}gripper_finger1_inner_knuckle_joint" type="continuous">
+            <parent link="${prefix}gripper_base_link"/>
+            <child link="${prefix}gripper_finger1_inner_knuckle_link"/>
             <axis xyz="0 0 1"/>
             <origin xyz="0.06142 0.0127 0" rpy="${pi} 0.0 0.0" />
             <limit lower="-3.14" upper="3.14" velocity="100.0" effort="0.1"/>
-            <mimic joint="${prefix}robotiq_85_left_knuckle_joint" offset="0"/>
-        </joint>
-        <joint name="${prefix}robotiq_85_right_inner_knuckle_joint" type="continuous">
-            <parent link="${prefix}robotiq_85_base_link"/>
-            <child link="${prefix}robotiq_85_right_inner_knuckle_link"/>
+            <mimic joint="${prefix}gripper_finger1_joint" offset="0"/>
+        </joint>
+        <joint name="${prefix}gripper_finger2_inner_knuckle_joint" type="continuous">
+            <parent link="${prefix}gripper_base_link"/>
+            <child link="${prefix}gripper_finger2_inner_knuckle_link"/>
             <axis xyz="0 0 1"/>
             <origin xyz="0.06142 -0.0127 0" rpy="0 0 0"/>
             <limit lower="-3.14" upper="3.14" velocity="100.0" effort="0.1"/>
-            <mimic joint="${prefix}robotiq_85_left_knuckle_joint" offset="0"/>
-        </joint>
-        <link name="${prefix}robotiq_85_left_inner_knuckle_link">
+            <mimic joint="${prefix}gripper_finger1_joint" offset="0"/>
+        </joint>
+        <link name="${prefix}gripper_finger1_inner_knuckle_link">
             <visual>
                 <geometry>
@@ -164,5 +198,12 @@
             </inertial>
         </link>
-        <link name="${prefix}robotiq_85_right_inner_knuckle_link">
+        <gazebo reference="${prefix}gripper_finger1_inner_knuckle_link">
+            <implicitSpringDamper>1</implicitSpringDamper>
+            <mu1>100000</mu1>
+            <mu2>100000</mu2>
+            <kp>100000000.0</kp>
+            <kd>1.0</kd>
+        </gazebo>
+        <link name="${prefix}gripper_finger2_inner_knuckle_link">
             <visual>
                 <geometry>
@@ -183,21 +224,28 @@
             </inertial>
         </link>
-        <joint name="${prefix}robotiq_85_left_finger_tip_joint" type="continuous">
-            <parent link="${prefix}robotiq_85_left_inner_knuckle_link"/>
-            <child link="${prefix}robotiq_85_left_finger_tip_link"/>
+        <gazebo reference="${prefix}gripper_finger2_inner_knuckle_link">
+            <implicitSpringDamper>1</implicitSpringDamper>
+            <mu1>100000</mu1>
+            <mu2>100000</mu2>
+            <kp>100000000.0</kp>
+            <kd>1.0</kd>
+        </gazebo>
+        <joint name="${prefix}gripper_finger1_finger_tip_joint" type="continuous">
+            <parent link="${prefix}gripper_finger1_inner_knuckle_link"/>
+            <child link="${prefix}gripper_finger1_finger_tip_link"/>
             <axis xyz="0 0 1"/>
             <origin xyz="0.04303959807 -0.03759940821 0.0" rpy="0.0 0.0 0.0"/>
             <limit lower="-3.14" upper="3.14" velocity="100.0" effort="0.1"/>
-            <mimic joint="${prefix}robotiq_85_left_knuckle_joint" multiplier="-1"/>
-        </joint>
-        <joint name="${prefix}robotiq_85_right_finger_tip_joint" type="continuous">
-            <parent link="${prefix}robotiq_85_right_inner_knuckle_link"/>
-            <child link="${prefix}robotiq_85_right_finger_tip_link"/>
+            <mimic joint="${prefix}gripper_finger1_joint" multiplier="-1"/>
+        </joint>
+        <joint name="${prefix}gripper_finger2_finger_tip_joint" type="continuous">
+            <parent link="${prefix}gripper_finger2_inner_knuckle_link"/>
+            <child link="${prefix}gripper_finger2_finger_tip_link"/>
             <axis xyz="0 0 1"/>
             <origin rpy="0.0 0.0 0.0" xyz="0.04303959807 -0.03759940821  0.0"/>
             <limit lower="-3.14" upper="3.14" velocity="100.0" effort="0.1"/>
-            <mimic joint="${prefix}robotiq_85_left_knuckle_joint" multiplier="-1"/>
-        </joint>
-        <link name="${prefix}robotiq_85_left_finger_tip_link">
+            <mimic joint="${prefix}gripper_finger1_joint" multiplier="-1"/>
+        </joint>
+        <link name="${prefix}gripper_finger1_finger_tip_link">
             <visual>
                 <geometry>
@@ -218,5 +266,12 @@
             </inertial>
         </link>
-        <link name="${prefix}robotiq_85_right_finger_tip_link">
+        <gazebo reference="${prefix}gripper_finger1_finger_tip_link">
+            <implicitSpringDamper>1</implicitSpringDamper>
+            <mu1>100000</mu1>
+            <mu2>100000</mu2>
+            <kp>100000000.0</kp>
+            <kd>1.0</kd>
+        </gazebo>
+        <link name="${prefix}gripper_finger2_finger_tip_link">
             <visual>
                 <geometry>
@@ -237,4 +292,11 @@
             </inertial>
         </link>
+        <gazebo reference="${prefix}gripper_finger2_finger_tip_link">
+            <implicitSpringDamper>1</implicitSpringDamper>
+            <mu1>100000</mu1>
+            <mu2>100000</mu2>
+            <kp>100000000.0</kp>
+            <kd>1.0</kd>
+        </gazebo>
         <xacro:robotiq_85_gripper_transmission prefix="${prefix}" />
     </xacro:macro>
